File: Shield carte avant/shield carte avant.brd (EAGLE design)
At the start: 68.6 x 53.3 mm, 29 parts, among them IC1 MCP2562-E_P, IC2 MCP2515-I_P, J1 22-05-7078-07, J2 22-05-7028-02, J3 22-05-7038-03, J5 22-05-7028-02, M1 ARDUINO_R3_ICSP

Commit message: Revue PJR
Parts:
- removed C1: 680 pF, rcl:C025-024X044
- added C7: 27pF, rcl:C025-030X050
- C5: value 680 pF -> 27pF; device rcl:C025-024X044 -> rcl:C025-030X050
- moved C5 27.1 mm to (36.5, 45.4)
- moved QUARTZ_16_MHZ1 2.86 mm to (44.8, 45.4)
- moved R1 2.31 mm to (20.3, 35.9)
- moved PS1 2.25 mm to (3.17, 34.0)
- moved R4 1.91 mm to (34.3, 27.6)
- moved SW2 1.59 mm to (34.3, 17.5)
- moved J5 1.42 mm to (13.8, 4.06)
- moved J2 1.27 mm to (5.08, 38.4)
- moved C3 0.90 mm to (25.1, 4.13)
- moved IC1 0.63 mm to (19.7, 43.2)
- moved R2 0.32 mm to (11.1, 43.2)
Connections:
- removed net N$2: R4.2, SW2.P$1
- removed net N$6: IC2.7, QUARTZ_16_MHZ1.2
- removed net RX: IC2.2
- removed net TX: IC2.1
- net +12V: no longer C1.1
- net +5V: no longer C1.2
- net GND: now also C7.1, PS1.5, SW2.P$2
- net N$3: now also IC2.8, QUARTZ_16_MHZ1.1; no longer PS1.5
- net N$7: now also C7.2, IC2.7, QUARTZ_16_MHZ1.2; no longer IC2.8, QUARTZ_16_MHZ1.1
- net RESET: now also R4.2, SW2.P$1; no longer SW2.P$2
- net RXD: now also IC2.2
- net TXD: now also IC2.1
Routing:
- net RXD: track 0.00 -> 38.3 mm
- net TXD: track 0.00 -> 35.7 mm
- net +5V: track 114.9 -> 92.0 mm
- net RESET: track 12.3 -> 24.2 mm
- net N$7: track 4.80 -> 13.7 mm
- net N$6: track 5.77 -> 0.00 mm
- net N$2: track 3.23 -> 0.00 mm
- net +12V: track 22.6 -> 19.6 mm
- net N$11: track 22.9 -> 21.0 mm
- net N$8: track 20.3 -> 18.8 mm
- net N$3: track 8.03 -> 9.54 mm
- net N$1: track 5.12 -> 3.79 mm

Commit message: Légères modifs avant envoie en prod
Parts:
- moved R4 7.43 mm to (41.3, 30.2), turned to 180 degrees
- moved J3 3.19 mm to (59.1, 43.5)
- moved IC2 2.54 mm to (34.3, 33.0)
- moved C10 1.27 mm to (28.9, 38.4)
- moved SW2 1.27 mm to (34.3, 16.2)
- moved C5 1.14 mm to (35.6, 44.8)
- moved QUARTZ_16_MHZ1 1.14 mm to (43.8, 44.8)
- moved C7 0.32 mm to (52.1, 44.8)
- moved C9 0.32 mm to (28.9, 44.5)
Connections:
- net SCL_SPI: now also J3.2; no longer J3.3
- net SDA_SPI: now also J3.1; no longer J3.2
- net TV: now also J3.3; no longer J3.1
Routing:
- net N$11: track 21.0 -> 8.73 mm
- net RESET: track 24.2 -> 31.8 mm
- net TV: track 7.18 -> 14.0 mm
- net SDA_SPI: track 10.8 -> 6.60 mm
- net SCL_SPI: track 14.4 -> 10.6 mm
- net SI: track 28.2 -> 31.1 mm
- net SCK: track 22.6 -> 25.1 mm
- net INT: track 31.3 -> 33.9 mm
- net SO: track 17.7 -> 20.0 mm
- net N$7: track 13.7 -> 15.0 mm
- net +5V: track 92.0 -> 90.8 mm
- net TXD: track 35.7 -> 34.7 mm
- net RXD: track 38.3 -> 38.9 mm
Other:
- board text added: "Dash 1"
- board text added: "RESET"
- board text removed: "Dashboard 1"
