File: Shield carte avant/shield carte avant.sch (EAGLE design)
At the start: 29 parts, among them IC1 MCP2562-E_P, IC2 MCP2515-I_P, J1 22-05-7078-07, J2 22-05-7028-02, J3 22-05-7038-03, J5 22-05-7028-02, M1 ARDUINO_R3_ICSP

Commit message: Légères modifs avant envoie en prod
Connections:
- net SCL_SPI: now also J3-2.S; no longer J3-3.S
- net SDA_SPI: now also J3-1.S; no longer J3-2.S
- net TV: now also J3-3.S; no longer J3-1.S
Changed lines of the file:
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@@
 </segment>
 <segment>
-<wire x1="68.58" y1="147.32" x2="55.88" y2="147.32" width="0.1524" layer="91"/>
-<label x="55.88" y="147.32" size="1.778" layer="95" rot="R180" xref="yes"/>
-<pinref part="J3" gate="-1" pin="S"/>
+<wire x1="68.58" y1="137.16" x2="55.88" y2="137.16" width="0.1524" layer="91"/>
+<label x="55.88" y="137.16" size="1.778" layer="95" rot="R180" xref="yes"/>
+<pinref part="J3" gate="-3" pin="S"/>
 </segment>
 </net>
@@
 </segment>
 <segment>
-<wire x1="68.58" y1="137.16" x2="55.88" y2="137.16" width="0.1524" layer="91"/>
-<label x="55.88" y="137.16" size="1.778" layer="95" rot="R180" xref="yes"/>
-<pinref part="J3" gate="-3" pin="S"/>
+<wire x1="68.58" y1="142.24" x2="55.88" y2="142.24" width="0.1524" layer="91"/>
+<label x="55.88" y="142.24" size="1.778" layer="95" rot="R180" xref="yes"/>
+<pinref part="J3" gate="-2" pin="S"/>
 </segment>
 </net>
@@
 </segment>
 <segment>
-<wire x1="68.58" y1="142.24" x2="55.88" y2="142.24" width="0.1524" layer="91"/>
-<label x="55.88" y="142.24" size="1.778" layer="95" rot="R180" xref="yes"/>
-<pinref part="J3" gate="-2" pin="S"/>
+<wire x1="68.58" y1="147.32" x2="55.88" y2="147.32" width="0.1524" layer="91"/>
+<label x="55.88" y="147.32" size="1.778" layer="95" rot="R180" xref="yes"/>
+<pinref part="J3" gate="-1" pin="S"/>
 </segment>
 </net>
